Commit message: fixed kinematic parameters + hardware parameters + fixed scanner position in robot model

File: robot_model/mp_500/mp_500.urdf.xacro (robot description, xacro)
@@ -155,5 +155,5 @@
 	<joint name="laserscanner_front_joint" type="fixed">
 		  <axis xyz="0 1 0" />
-		  <origin xyz="0.230 0 0.110" rpy="3.14 0 0" />
+		  <origin xyz="0.244 0 0.141" rpy="3.14 0 0" />
 		  <parent link="base_link"/>
 		  <child link="laserscanner_front_link"/>

Commit message: added robot body

File: robot_model/mp_500/mp_500.urdf.xacro (robot description, xacro)
@@ -47,5 +47,5 @@
 		<origin xyz="0.0 0.0 0.0" rpy="0 0 1.57" /><!-- for STL -->
         <geometry>
-            <mesh filename="package://neo_mp_500/robot_model/mp_500/meshes/MP-400-BODY.STL" scale="0.001 0.001 0.001"/>
+            <mesh filename="package://neo_mp_500/robot_model/mp_500/meshes/MP-500-BODY.STL" scale="0.001 0.001 0.001"/>
 	    	<!--cylinder length="0.381" radius="0.2545"/-->
 	    	<!--box size="0.445 0.277 0.17"/-->
@@ -180,31 +180,3 @@
 	  	</collision>
 	</link>
-        <!--+++++++++++++++++++laserscanner_back_joint++++++++++++++++++++++++-->
-        <joint name="laserscanner_back_joint" type="fixed">
-                  <axis xyz="0 1 0" />
-                  <origin xyz="-0.354 0 0.110" rpy="3.14 0 3.14" />
-                  <parent link="base_link"/>
-                  <child link="laserscanner_back_link"/>
-        </joint>
-        <!--+++++++++++++++++++laserscanner_back_link++++++++++++++++++++++++-->
-        <link name="laserscanner_back_link" type="laser">
-                <inertial>
-                        <mass value="0.001" />
-                        <origin xyz="0 0 0" rpy="0 0 0" />
-                        <inertia ixx="0.0001" ixy="0" ixz="0" iyy="0.000001" iyz="0" izz="0.0001" />
-                </inertial>
-                <visual>
-                        <origin xyz="0 0 0" rpy="0 0 -1.57" />
-                        <geometry>
-                                <mesh filename="package://neo_mp_500/robot_model/mp_500/meshes/SICK-S300.STL" />
-                        </geometry>
-                        <material name="Neobotix/Yellow" />
-                </visual>
-                <collision>
-                        <origin xyz="0 0 0" rpy="0 0 0" />
-                        <geometry>
-                        <cylinder length="0.154" radius="0.053" />
-                        </geometry>
-                </collision>
-        </link>
 </robot>

Commit message: fixed robot model scaling

File: robot_model/mp_500/mp_500.urdf.xacro (robot description, xacro)
@@ -47,5 +47,5 @@
 		<origin xyz="0.0 0.0 0.0" rpy="0 0 1.57" /><!-- for STL -->
         <geometry>
-            <mesh filename="package://neo_mp_500/robot_model/mp_500/meshes/MP-500-BODY.STL" scale="0.001 0.001 0.001"/>
+            <mesh filename="package://neo_mp_500/robot_model/mp_500/meshes/MP-500-BODY.STL" scale="1 1 1"/>
 	    	<!--cylinder length="0.381" radius="0.2545"/-->
 	    	<!--box size="0.445 0.277 0.17"/-->

Commit message: updated robot model and added .launch file

File: robot_model/mp_500/mp_500.urdf.xacro (robot description, xacro)
@@ -45,7 +45,7 @@
       <visual name='body'>
         <!--origin xyz="0.0 0.0 0.234" rpy="0 0 1.57" /--><!-- for cylinder -->
-		<origin xyz="0.0 0.0 0.0" rpy="0 0 1.57" /><!-- for STL -->
+		<origin xyz="0.0 0.0 0.08" rpy="0 0 1.57" /><!-- for STL -->
         <geometry>
-            <mesh filename="package://neo_mp_500/robot_model/mp_500/meshes/MP-500-BODY.STL" scale="1 1 1"/>
+            <mesh filename="package://neo_mp_500/robot_model/mp_500/meshes/MP-500-BODY.STL" scale="0.01 0.01 0.01"/>
 	    	<!--cylinder length="0.381" radius="0.2545"/-->
 	    	<!--box size="0.445 0.277 0.17"/-->
@@ -56,6 +56,6 @@
         <origin xyz="0.0 0.0 0.234" rpy="0 0 0" />
         <geometry>
-          <!--box size="0.445 0.277 0.17"/-->
-          <cylinder length="0.381" radius="0.2545"/>
+          <box size="0.830 0.600 0.400"/>
+          <!--cylinder length="0.381" radius="0.2545"/-->
         </geometry>
       </collision>
@@ -97,12 +97,11 @@
       <inertia ixx="0.0051" ixy="0" ixz="0" iyy="0.0051" iyz="0" izz="0.009" />
     </inertial>
-    <visual>
+    <!--visual>
      	<origin xyz="0.0 0.0 -0.016" rpy="0 0 0" />
      	<geometry>
-        	<!--mesh filename="package://neo_robot_descriptions/mp_400/meshes/MP-400-WHEEL.STL" scale="0.001 0.001 0.001"/-->
 			<cylinder radius="0.075" length="0.03"/>
      	</geometry>
      	<material name="Neobotix/Black" />
-    </visual>
+    </visual-->
     <collision>
      	<origin xyz="0.0 0.0 -0.016" rpy="0 0 0" />
@@ -128,12 +127,11 @@
 		  <inertia ixx="0.0051" ixy="0" ixz="0" iyy="0.0051" iyz="0" izz="0.009" />
 		</inertial>
-		<visual>
+		<!--visual>
 		 	<origin xyz="0 0.0 0.016" rpy="0 0 0" />
 		 	<geometry>
-		    	<!--mesh filename="package://neo_robot_descriptions/mp_400/meshes/MP-400-WHEEL.STL" scale="0.001 0.001 0.001"/-->
 				<cylinder radius="0.075" length="0.03"/>
 		 	</geometry>
 		 	<material name="Neobotix/Black" />
-		</visual>
+		</visual-->
 		<collision>
 		 	<origin xyz="0.0 0.0 0.016" rpy="0 0 0" />
@@ -163,9 +161,9 @@
 		<inertial>
 			<mass value="0.001" />
-			<origin xyz="0 0 0" rpy="0 0 0" />
+			<origin xyz="0 0 0.0" rpy="0 0 0" />
 			<inertia ixx="0.0001" ixy="0" ixz="0" iyy="0.000001" iyz="0" izz="0.0001" />
 	  	</inertial>
 	  	<visual>
-			<origin xyz="0 0 0" rpy="0 0 -1.57" />
+			<origin xyz="0 0 -0.04" rpy="0 0 -1.57" />
 			<geometry>
 		  		<mesh filename="package://neo_mp_500/robot_model/mp_500/meshes/SICK-S300.STL" />

Commit message: new and more detalied robot model

File: robot_model/mp_500/mp_500.urdf.xacro (robot description, xacro)
@@ -2,179 +2,29 @@
 <!-- Materials -->
 <robot xmlns:xacro="http://www.ros.org/wiki/xacro" name="mp_500">
-	<material name="Neobotix/Black">
-        <color rgba="0.0 0.0 0.0 1.0"/>
-    </material>
-    <material name="Neobotix/Blue">
-        <color rgba="0.0 0.0 0.8 1.0"/>
-    </material>
-    <material name="Neobotix/Green">
-        <color rgba="0.0 0.8 0.0 1.0"/>
-    </material>
-    <material name="Neobotix/Grey">
-        <color rgba="0.7 0.7 0.7 1.0"/>
-    </material>
-    <material name="Neobotix/Grey2">
-        <color rgba="0.9 0.9 0.9 1.0"/>
-    </material>
-    <material name="Neobotix/Red">
-        <color rgba="0.8 0.0 0.0 1.0"/>
-    </material>
-    <material name="Neobotix/White">
-        <color rgba="1.0 1.0 1.0 1.0"/>
-    </material>
-    <material name="Neobotix/Yellow">
-        <color rgba="1.0 1.0 0 10" />
-    </material>
+<xacro:include filename="$(find neo_mp_500)/robot_model/mp_500/xacros/mp_500_gazebo.xacro" />
 <!--++++++++++++++++++++++++++++++base_link++++++++++++++++++++++++++++++++++++++++++++++++++++-->
 <!--++++++++++++++++++++body++++++++++++++++++++++++++++-->
-	<link name="base_link">
-      <!--inertial>
-        <mass value="67.010" />
-        <origin xyz="0.0 0.0 0.234" rpy="0 0 0"/>
-        <inertia ixx="1417853.715" ixy="17813.155" ixz="-21078.206"
-                 iyy="2030191.708" iyz="-4813.295"
-                 izz="2180211.662" />
-      </inertial-->
-	  <inertial>
-		  <mass value="5.67" />
-		    <origin xyz="0 0 0.0" rpy="0 0 0"/>
-		    <inertia ixx="0.07" ixy="0.0" ixz="0.0"
-		             iyy="0.08" iyz="0.0"
-		             izz="0.1" />
-	  </inertial>
-      <visual name='body'>
-        <!--origin xyz="0.0 0.0 0.234" rpy="0 0 1.57" /--><!-- for cylinder -->
-		<origin xyz="0.0 0.0 0.08" rpy="0 0 1.57" /><!-- for STL -->
-        <geometry>
-            <mesh filename="package://neo_mp_500/robot_model/mp_500/meshes/MP-500-BODY.STL" scale="0.01 0.01 0.01"/>
-	    	<!--cylinder length="0.381" radius="0.2545"/-->
-	    	<!--box size="0.445 0.277 0.17"/-->
-        </geometry>
-        <material name="Neobotix/Grey" />
-      </visual>
-      <collision name='body_collision'>
-        <origin xyz="0.0 0.0 0.234" rpy="0 0 0" />
-        <geometry>
-          <box size="0.830 0.600 0.400"/>
-          <!--cylinder length="0.381" radius="0.2545"/-->
-        </geometry>
-      </collision>
-<!--+++++++++++++++++++castor_front++++++++++++++++++++++++-->
-	<visual name='castor_front_visual'>
-          <origin xyz="0.2 0 0.018" rpy="0 0 0" />
-          <geometry>
-            <sphere radius="0.016"/>
-          </geometry>
-          <material name="Neobotix/Black" />
-      </visual>
-      <collision name='castor_front_collision'>
-	  	<origin xyz="0.2 0 0.018 " rpy="0 0 0" />
-          <geometry>
-            <sphere radius="0.016"/>
-          </geometry>
-    </collision>
-<!--+++++++++++++++++++castor_back++++++++++++++++++++++++-->
-	<visual name='castor_back_visual'>
-          <origin xyz="-0.2 0 0.018" rpy="0 0 0" />
-          <geometry>
-            <sphere radius="0.016"/>
-          </geometry>
-          <material name="Neobotix/Black" />
-      </visual>
-      <collision name='castor_back_collision'>
-	  	<origin xyz="-0.2 0 0.018 " rpy="0 0 0" />
-          <!--pose>0.3 0 -0.12 0 -0 0</pose-->
-          <geometry>
-            <sphere radius="0.016"/>
-          </geometry>
-       </collision>
-    </link>
-<!--+++++++++++++++++++wheel_left_link++++++++++++++++++++++++-->
-<link name="wheel_left_link" type="wheel">
-    <inertial>
-      <mass value="1.5" />
-      <origin xyz="0.0 0.0 -0.016" rpy="0 0 0" />
-      <inertia ixx="0.0051" ixy="0" ixz="0" iyy="0.0051" iyz="0" izz="0.009" />
-    </inertial>
-    <!--visual>
-     	<origin xyz="0.0 0.0 -0.016" rpy="0 0 0" />
-     	<geometry>
-			<cylinder radius="0.075" length="0.03"/>
-     	</geometry>
-     	<material name="Neobotix/Black" />
-    </visual-->
-    <collision>
-     	<origin xyz="0.0 0.0 -0.016" rpy="0 0 0" />
-     	<geometry>
-        	<cylinder radius="0.075" length="0.03"/>
-     	</geometry>
-    </collision>
-</link>
-<!--+++++++++++++++++++wheel_left_joint++++++++++++++++++++++++-->
-	<joint name="wheel_left_joint" type="revolute">
-		<origin xyz="0 -0.2645 0.075" rpy="0 1.57 1.57" />
-    	<axis xyz="0 0 1"/>
-    	<limit effort="1000.0" lower="-1e+16" upper="1e+16" velocity="3.5"/>
-    	<joint_properties damping="0.0" friction="0.0" />
-    	<parent link="base_link" />
-    	<child link="wheel_left_link" />
-    </joint>
-	<!--+++++++++++++++++++wheel_right_link++++++++++++++++++++++++-->
-	<link name="wheel_right_link" type="wheel">
-		<inertial>
-		  <mass value="1.5" />
-		  <origin xyz="0 0.0 0.016" rpy="0 0 0" />
-		  <inertia ixx="0.0051" ixy="0" ixz="0" iyy="0.0051" iyz="0" izz="0.009" />
-		</inertial>
-		<!--visual>
-		 	<origin xyz="0 0.0 0.016" rpy="0 0 0" />
-		 	<geometry>
-				<cylinder radius="0.075" length="0.03"/>
-		 	</geometry>
-		 	<material name="Neobotix/Black" />
-		</visual-->
-		<collision>
-		 	<origin xyz="0.0 0.0 0.016" rpy="0 0 0" />
-		 	<geometry>
-		    	<cylinder radius="0.075" length="0.03"/>
-		 	</geometry>
-		</collision>
-	</link>
-	<!--+++++++++++++++++++wheel_right_joint++++++++++++++++++++++++-->
-	<joint name="wheel_right_joint" type="revolute">
-    	<origin xyz="0 0.2645 0.075" rpy="0 1.57 1.57" />
-    	<axis xyz="0 0 1"/>
-    	<limit effort="1000.0" lower="-1e+16" upper="1e+16" velocity="3.5"/>
-    	<joint_properties damping="0.0" friction="0.0" />
-    	<parent link="base_link" />
-    	<child link="wheel_right_link" />
-    </joint>
-	<!--+++++++++++++++++++laserscanner_front_joint++++++++++++++++++++++++-->
-	<joint name="laserscanner_front_joint" type="fixed">
-		  <axis xyz="0 1 0" />
-		  <origin xyz="0.244 0 0.141" rpy="3.14 0 0" />
-		  <parent link="base_link"/>
-		  <child link="laserscanner_front_link"/>
-	</joint>
-	<!--+++++++++++++++++++laserscanner_front_link++++++++++++++++++++++++-->
-	<link name="laserscanner_front_link" type="laser">
-		<inertial>
-			<mass value="0.001" />
-			<origin xyz="0 0 0.0" rpy="0 0 0" />
-			<inertia ixx="0.0001" ixy="0" ixz="0" iyy="0.000001" iyz="0" izz="0.0001" />
-	  	</inertial>
-	  	<visual>
-			<origin xyz="0 0 -0.04" rpy="0 0 -1.57" />
-			<geometry>
-		  		<mesh filename="package://neo_mp_500/robot_model/mp_500/meshes/SICK-S300.STL" />
-			</geometry>
-			<material name="Neobotix/Yellow" />
-	  	</visual>
-	  	<collision>
-			<origin xyz="0 0 0" rpy="0 0 0" />
-			<geometry>
-		  	<cylinder length="0.154" radius="0.053" />
-			</geometry>
-	  	</collision>
-	</link>
+<xacro:include filename="$(find neo_mp_500)/robot_model/mp_500/xacros/mp_500_body.xacro" />
+<!--+++++++++++++++++++castor_wheel_link++++++++++++++++++++++++-->
+<xacro:include filename="$(find neo_mp_500)/robot_model/mp_500/xacros/mp_500_caster_wheel.xacro" />
+<!--+++++++++++++++++++left_wheel_link++++++++++++++++++++++++-->
+<xacro:include filename="$(find neo_mp_500)/robot_model/mp_500/xacros/mp_500_fixed_wheel.xacro" />
+  <xacro:mp_500_base name="base_link">
+  </xacro:mp_500_base>
+  <!-- Wheel Macro -->
+  <xacro:caster_wheel name="wheel_front" parent="base_link">
+    <origin xyz="-0.37 0. 0.06" rpy="-1.570796 0 1.57" />
+  </xacro:caster_wheel>
+  <xacro:fixed_wheel name="fixed_wheel_right" parent="base_link">
+    <origin xyz="0. -0.25 0.12" rpy="0 0 -1.570796" />
+  </xacro:fixed_wheel>
+  <xacro:fixed_wheel name="fixed_wheel_left" parent="base_link">
+    <origin xyz="0. 0.25 0.12" rpy="0 0 -1.570796" />
+  </xacro:fixed_wheel>
+ <!--+++++++++++++++++++laserscanner_front_link++++++++++++++++++++++++-->
+   <!-- SENSORS -->
+  <xacro:include filename="$(find neo_mp_500)/robot_model/mp_500/xacros/sick_laser.xacro" />
+  <xacro:sick_laser_v0 name="laserscanner" parent="base_link" ros_topic="sick_300/scan">
+    <origin xyz="0.244 0 0.141" rpy="0 0 0" />
+  </xacro:sick_laser_v0>
 </robot>

Commit message: fixed frame names and locations

File: robot_model/mp_500/mp_500.urdf.xacro (robot description, xacro)
@@ -11,20 +11,20 @@
 <xacro:include filename="$(find neo_mp_500)/robot_model/mp_500/xacros/mp_500_fixed_wheel.xacro" />
   <xacro:mp_500_base name="base_link">
-  </xacro:mp_500_base>
-  <!-- Wheel Macro -->
-  <xacro:caster_wheel name="wheel_front" parent="base_link">
-    <origin xyz="-0.37 0. 0.06" rpy="-1.570796 0 1.57" />
-  </xacro:caster_wheel>
-  <xacro:fixed_wheel name="fixed_wheel_right" parent="base_link">
-    <origin xyz="0. -0.25 0.12" rpy="0 0 -1.570796" />
-  </xacro:fixed_wheel>
-  <xacro:fixed_wheel name="fixed_wheel_left" parent="base_link">
-    <origin xyz="0. 0.25 0.12" rpy="0 0 -1.570796" />
-  </xacro:fixed_wheel>
- <!--+++++++++++++++++++laserscanner_front_link++++++++++++++++++++++++-->
-   <!-- SENSORS -->
-  <xacro:include filename="$(find neo_mp_500)/robot_model/mp_500/xacros/sick_laser.xacro" />
-  <xacro:sick_laser_v0 name="laserscanner" parent="base_link" ros_topic="sick_300/scan">
-    <origin xyz="0.244 0 0.141" rpy="0 0 0" />
-  </xacro:sick_laser_v0>
+</xacro:mp_500_base>
+<!-- Wheel Macro -->
+<xacro:caster_wheel name="caster_wheel" parent="base_link">
+	<origin xyz="-0.43 0. 0.171" rpy="-1.570796 0 1.570796 " />
+</xacro:caster_wheel>
+<xacro:fixed_wheel name="wheel_right" parent="base_link">
+	<origin xyz="0. -0.25 0.125" rpy="0 0 1.570796" />
+</xacro:fixed_wheel>
+<xacro:fixed_wheel name="wheel_left" parent="base_link">
+	<origin xyz="0. 0.25 0.125" rpy="0 0 -1.570796" />
+</xacro:fixed_wheel>
+<!--+++++++++++++++++++laserscanner_front_link++++++++++++++++++++++++-->
+<!-- SENSORS -->
+<xacro:include filename="$(find neo_mp_500)/robot_model/mp_500/xacros/sick_laser.xacro" />
+<xacro:sick_laser_v0 name="laserscanner_1" parent="base_link" ros_topic="sick/scan">
+	<origin xyz="0.244 0 0.141" rpy="3.14 0 0" />
+</xacro:sick_laser_v0>
 </robot>

File: robot_model/mp_500/xacros/mp_500_body.xacro (robot description, xacro)
@@ -11,5 +11,5 @@
   </inertial>
   <visual name='body'>
-  <origin xyz="0.0 0.0 -0.06" rpy="0 0 1.570796" /><!-- for STL -->
+  <origin xyz="0.0 0.0 0" rpy="0 0 1.570796" />
   <geometry>
       <mesh filename="package://neo_mp_500/robot_model/mp_500/meshes/MP-500-BODY.dae" scale="0.001 0.001 0.001"/>

File: robot_model/mp_500/xacros/mp_500_caster_wheel.xacro (robot description, xacro)
@@ -16,5 +16,5 @@
     </inertial>
       <visual name='castor_wheel'>
-    <origin xyz="0.0 -0.06 0.06" rpy="0 0 0" />
+    <origin xyz="0 0 0" rpy="0 0 0" />
         <geometry>
             <mesh filename="package://neo_mp_500/robot_model/mp_500/meshes/MP-500-WHEEL.dae" scale="0.001 0.001 0.001"/>
@@ -24,5 +24,5 @@
       <origin xyz="0 0 0" rpy="0 0 0" />
       <geometry>
-            <mesh filename="package://neo_mp_500/robot_model/mp_500/meshes/MP-500-WHEEL.STL" scale="0.001 0.001 0.001"/>
+            <mesh filename="package://neo_mp_500/robot_model/mp_500/meshes/MP-500-WHEEL.dae" scale="0.001 0.001 0.001"/>
       </geometry>
     </collision>

File: robot_model/mp_500/xacros/mp_500_fixed_wheel.xacro (robot description, xacro)
@@ -16,5 +16,5 @@
     </inertial>
       <visual>
-    <origin xyz="0 0. -0.04" rpy=" 0 0 0" />
+    <origin xyz="0 0 0" rpy="0 0 0" />
         <geometry>
             <mesh filename="package://neo_mp_500/robot_model/mp_500/meshes/MP-500-FIXED-WHEEL.dae" scale="0.001 0.001 0.001"/>
@@ -24,5 +24,5 @@
      <origin xyz="0 0 0" rpy="0 0 0" />
       <geometry>
-            <mesh filename="package://neo_mp_500/robot_model/mp_500/meshes/MP-500-WHEEL.STL" scale="0.001 0.001 0.001"/>
+            <mesh filename="package://neo_mp_500/robot_model/mp_500/meshes/MP-500-FIXED-WHEEL.dae" scale="0.001 0.001 0.001"/>
       </geometry>
     </collision>

File: robot_model/mp_500/xacros/mp_500_gazebo.xacro (robot description, xacro)
@@ -9,6 +9,6 @@
     <self_collide>false</self_collide>
   </gazebo>
-  <gazebo reference="laserscanner_link">
-      <sensor type="ray" name="laserscanner_link">
+  <gazebo reference="laserscanner_1_link">
+      <sensor type="ray" name="laserscanner_1_link">
           <pose>0 0 0 0 0 0</pose>
           <visualize>true</visualize>
@@ -38,7 +38,7 @@
             </noise>
           </ray>
-          <plugin name="laserscanner_link" filename="libgazebo_ros_laser.so">
-            <topicName>sick_s300/scan</topicName>
-            <frameName>laserscanner_link</frameName>
+          <plugin name="laserscanner_1_link" filename="libgazebo_ros_laser.so">
+            <topicName>sick/scan</topicName>
+            <frameName>laserscanner_1_link</frameName>
           </plugin>
         </sensor>

File: robot_model/mp_500/xacros/sick_laser.xacro (robot description, xacro)
@@ -16,5 +16,5 @@
       <visual>
       <!-- SICK S3 sensor: Uncomment/Comment it out if required  -->
-      <origin xyz="0 0 0.12" rpy="1.57 0 3.14" />
+      <origin xyz="0 0 -0.12" rpy="-1.57 0 3.14" />
         <geometry>
         <mesh filename="package://neo_mp_500/robot_model/mp_500/meshes/SICK-S300.dae" scale="0.001 0.001 0.001" />
@@ -22,5 +22,5 @@
       </visual>
       <collision>
-        <origin xyz="0 0 0" rpy="1.57 0 3.14" />
+        <origin xyz="0 0 -0.13" rpy="-1.57 0 3.14" />
         <geometry>
         <mesh filename="package://neo_mp_500/robot_model/mp_500/meshes/SICK-S300.dae" scale="0.001 0.001 0.001" />
@@ -28,13 +28,13 @@
       </collision>
       <!-- Microscan 3 sensor: Uncomment/Comment it out if required  -->
-<!--  <origin xyz="-0.0 0 0.06" rpy="-1.57 0 0" />
+<!--  <origin xyz="-0.0 0 -0.06" rpy="1.57 0 0" />
       <geometry>
-      <mesh filename="package://neo_simulation/robots/mp_500/meshes/SICK-MICROSCAN3.dae" scale="0.001 0.001 0.001" />
+      <mesh filename="package://neo_mp_500/robot_model/mp_500/meshes/SICK-MICROSCAN3.dae" scale="0.001 0.001 0.001" />
       </geometry>
       </visual>
       <collision>
- <origin xyz="-0.0 0 0.06" rpy="-1.57 0 0" />
+ <origin xyz="-0.0 0 -0.06" rpy="1.57 0 0" />
       <geometry>
-        <mesh filename="package://neo_simulation/robots/mp_500/meshes/SICK-MICROSCAN3.dae" scale="0.001 0.001 0.001" />
+        <mesh filename="package://neo_mp_500/robot_model/mp_500/meshes/SICK-MICROSCAN3.dae" scale="0.001 0.001 0.001" />
         </geometry>
       </collision> -->

Commit message: changed name for laser scanner from laser to lidar

File: robot_model/mp_500/mp_500.urdf.xacro (robot description, xacro)
@@ -25,6 +25,6 @@
 <!-- SENSORS -->
 <xacro:include filename="$(find neo_mp_500)/robot_model/mp_500/xacros/sick_laser.xacro" />
-<xacro:sick_laser_v0 name="laser_1" parent="base_link" ros_topic="sick/scan">
+<xacro:sick_lidar_v0 name="lidar_1" parent="base_link" ros_topic="sick/scan">
 	<origin xyz="0.244 0 0.141" rpy="3.14 0 0" />
-</xacro:sick_laser_v0>
+</xacro:sick_lidar_v0>
 </robot>

File: robot_model/mp_500/xacros/mp_500_gazebo.xacro (robot description, xacro)
@@ -9,6 +9,6 @@
     <self_collide>false</self_collide>
   </gazebo>
-  <gazebo reference="laser_1_link">
-      <sensor type="ray" name="laserscanner_1_link">
+  <gazebo reference="lidar_1_link">
+      <sensor type="ray" name="lidar_1_link">
           <pose>0 0 0 0 0 0</pose>
           <visualize>true</visualize>
@@ -38,5 +38,5 @@
             </noise>
           </ray>
-          <plugin name="laserscanner_1_link" filename="libgazebo_ros_laser.so">
+          <plugin name="lidar_1_link" filename="libgazebo_ros_laser.so">
             <topicName>sick/scan</topicName>
             <frameName>laserscanner_1_link</frameName>

File: robot_model/mp_500/xacros/sick_laser.xacro (robot description, xacro)
@@ -1,5 +1,5 @@
 <?xml version="1.0"?>
 <robot xmlns:xacro="http://www.ros.org/wiki/xacro" name="mp_500">
-  <xacro:macro name="sick_laser_v0" params="name parent *origin ros_topic">
+  <xacro:macro name="sick_lidar_v0" params="name parent *origin ros_topic">
     <joint name="${name}_joint" type="fixed">
       <axis xyz="0 1 0" />
