Commit message: robot models are updated

File: robot_model/mp_500/mp_500.urdf.xacro (robot description, xacro)
@@ -1,30 +1,113 @@
 <?xml version="1.0"?>
-<!-- Materials -->
 <robot xmlns:xacro="http://www.ros.org/wiki/xacro" name="mp_500">
-<xacro:include filename="$(find neo_mp_500)/robot_model/mp_500/xacros/mp_500_gazebo.xacro" />
-<!--++++++++++++++++++++++++++++++base_link++++++++++++++++++++++++++++++++++++++++++++++++++++-->
-<!--++++++++++++++++++++body++++++++++++++++++++++++++++-->
-<xacro:include filename="$(find neo_mp_500)/robot_model/mp_500/xacros/mp_500_body.xacro" />
-<!--+++++++++++++++++++castor_wheel_link++++++++++++++++++++++++-->
-<xacro:include filename="$(find neo_mp_500)/robot_model/mp_500/xacros/mp_500_caster_wheel.xacro" />
-<!--+++++++++++++++++++left_wheel_link++++++++++++++++++++++++-->
-<xacro:include filename="$(find neo_mp_500)/robot_model/mp_500/xacros/mp_500_fixed_wheel.xacro" />
+  <xacro:include filename="$(find neo_mp_500)/robot_model/mp_500/xacros/mp_500_gazebo.xacro" />
+  <!--++++++++++++++++++++++++++++++base_link++++++++++++++++++++++++++++++++++++++++++++++++++++-->
+  <!--++++++++++++++++++++body++++++++++++++++++++++++++++-->
+  <xacro:include filename="$(find neo_mp_500)/robot_model/mp_500/xacros/mp_500_body.xacro" />
+  <!--+++++++++++++++++++castor_wheel_link++++++++++++++++++++++++-->
+  <xacro:include filename="$(find neo_mp_500)/robot_model/mp_500/xacros/mp_500_caster_wheel.xacro" />
+  <!--+++++++++++++++++++left_wheel_link++++++++++++++++++++++++-->
+  <xacro:include filename="$(find neo_mp_500)/robot_model/mp_500/xacros/mp_500_fixed_wheel_left.xacro" />
+  <xacro:include filename="$(find neo_mp_500)/robot_model/mp_500/xacros/mp_500_fixed_wheel_right.xacro" />
+  <!-- SENSORS -->
+  <!-- Sick S300 - Comment/Uncomment if required  -->
+  <xacro:include filename="$(find neo_mp_500)/robot_model/mp_500/xacros/sick_S300.xacro" />
+  <!-- Microscan - Comment/Uncomment if required -->
+  <!-- <xacro:include filename="$(find neo_mp_500)/robot_model/mp_500/xacros/micro_scan.xacro" /> -->
+  <!-- USS and IMU - Comment/Uncomment if required  -->
+  <!-- <xacro:include filename="$(find neo_mp_500)/robot_model/mp_500/xacros/imu.xacro" />
+  <xacro:include filename="$(find neo_mp_500)/robot_model/mp_500/xacros/ultrasonic.xacro" /> -->
   <xacro:mp_500_base name="base_link">
-</xacro:mp_500_base>
-<!-- Wheel Macro -->
-<xacro:caster_wheel name="caster_wheel" parent="base_link">
-	<origin xyz="-0.43 0. 0.171" rpy="-1.570796 0 1.570796 " />
-</xacro:caster_wheel>
-<xacro:fixed_wheel name="wheel_right" parent="base_link">
-	<origin xyz="0. -0.25 0.125" rpy="0 0 1.570796" />
-</xacro:fixed_wheel>
-<xacro:fixed_wheel name="wheel_left" parent="base_link">
-	<origin xyz="0. 0.25 0.125" rpy="0 0 -1.570796" />
-</xacro:fixed_wheel>
-<!--+++++++++++++++++++laserscanner_front_link++++++++++++++++++++++++-->
-<!-- SENSORS -->
-<xacro:include filename="$(find neo_mp_500)/robot_model/mp_500/xacros/sick_laser.xacro" />
-<xacro:sick_lidar_v0 name="lidar_1" parent="base_link" ros_topic="sick/scan">
-	<origin xyz="0.244 0 0.141" rpy="3.14 0 0" />
-</xacro:sick_lidar_v0>
+  </xacro:mp_500_base>
+  <!-- Wheel Macro -->
+  <xacro:caster_wheel name="caster_wheel" parent="base_link">
+    <origin xyz="-0.43 0. 0.176" rpy="-1.570796 0 1.570796 " />
+  </xacro:caster_wheel>
+  <xacro:fixed_wheel_right name="wheel_right" parent="base_link" number="1">
+    <origin xyz="0. -0.25 0.13" rpy="0 0 -1.570796" />
+  </xacro:fixed_wheel_right>
+  <xacro:fixed_wheel_left name="wheel_left" parent="base_link" number="2">
+    <origin xyz="0. 0.25 0.13" rpy="0 0 -1.570796" />
+  </xacro:fixed_wheel_left>
+ <!--+++++++++++++++++++laserscanner_front_link++++++++++++++++++++++++-->
+   <!-- SENSORS -->
+  <xacro:sick_laser_v0 name="lidar_1" parent="base_link" ros_topic="lidar_1/scan_filtered">
+    <origin xyz="0.244 0 0.141" rpy="3.14 0 0" />
+  </xacro:sick_laser_v0>
+     <!--+++++++++++++++++++ IMU ++++++++++++++++++++++++-->
+ <!-- Comment or uncomment based on your requirement -->
+<!--   <xacro:imu name="imu_1" parent="base_link">
+    <origin xyz="0.100 0 0.300" rpy="0 0 3.14" />
+  </xacro:imu> -->
+  <!--+++++++++++++++++++ Ultra Sonic ++++++++++++++++++++++++-->
+  <!-- Comment or uncomment based on your requirement -->
+  <!-- SENSOR 1 -->
+  <!-- xacro:us_sensor name="us_1" parent="base_link">
+    <origin xyz="0.100 0 0.300" rpy="0 3.14 3.14" />
+  </xacro:us_sensor-->
+  <!-- SENSOR 2 -->
+  <!-- xacro:us_sensor name="us_2" parent="base_link">
+    <origin xyz="0.110 0 0.300" rpy="0 3.14 3.14" />
+  </xacro:us_sensor-->
+  <!-- SENSOR 3 -->
+  <!-- xacro:us_sensor name="us_3" parent="base_link">
+    <origin xyz="0.120 0 0.300" rpy="0 3.14 3.14" />
+  </xacro:us_sensor-->
+  <!-- SENSOR 4 -->
+  <!-- xacro:us_sensor name="us_4" parent="base_link">
+    <origin xyz="0.130 0 0.300" rpy="0 3.14 3.14" />
+  </xacro:us_sensor-->
+  <!-- SENSOR 5 -->
+  <!-- xacro:us_sensor name="us_5" parent="base_link">
+    <origin xyz="0.140 0 0.300" rpy="0 3.14 3.14" />
+  </xacro:us_sensor-->
+  <!-- SENSOR 6 -->
+  <!-- xacro:us_sensor name="us_6" parent="base_link">
+    <origin xyz="0.150 0 0.300" rpy="0 3.14 3.14" />
+  </xacro:us_sensor-->
+  <!-- SENSOR 7 -->
+  <!-- xacro:us_sensor name="us_7" parent="base_link">
+    <origin xyz="0.160 0 0.300" rpy="0 3.14 3.14" />
+  </xacro:us_sensor-->
+  <!-- SENSOR 8 -->
+  <!-- xacro:us_sensor name="us_8" parent="base_link">
+    <origin xyz="0.170 0 0.300" rpy="0 3.14 3.14" />
+  </xacro:us_sensor-->
+  <!-- SENSOR 9 -->
+  <!-- xacro:us_sensor name="us_9" parent="base_link">
+    <origin xyz="0.180 0 0.300" rpy="0 3.14 3.14" />
+  </xacro:us_sensor-->
+  <!-- SENSOR 10 -->
+  <!-- xacro:us_sensor name="us_10" parent="base_link">
+    <origin xyz="0.100 0 0.300" rpy="0 3.14 3.14" />
+  </xacro:us_sensor-->
+  <!-- SENSOR 11 -->
+  <!-- xacro:us_sensor name="us_11" parent="base_link">
+    <origin xyz="0.100 0 0.300" rpy="0 3.14 3.14" />
+  </xacro:us_sensor-->
+  <!-- SENSOR 12 -->
+  <!-- xacro:us_sensor name="us_12" parent="base_link">
+    <origin xyz="0.190 0 0.300" rpy="0 3.14 3.14" />
+  </xacro:us_sensor-->
+  <!-- SENSOR 13 -->
+  <!-- xacro:us_sensor name="us_13" parent="base_link">
+    <origin xyz="0.200 0 0.300" rpy="0 3.14 3.14" />
+  </xacro:us_sensor-->
+  <!-- SENSOR 14 -->
+  <!-- xacro:us_sensor name="us_14" parent="base_link">
+    <origin xyz="0.210 0 0.300" rpy="0 3.14 3.14" />
+  </xacro:us_sensor-->
+  <!-- SENSOR 15 -->
+  <!-- xacro:us_sensor name="us_15" parent="base_link">
+    <origin xyz="0.220 0 0.300" rpy="0 3.14 3.14" />
+  </xacro:us_sensor-->
+  <!-- SENSOR 16 -->
+  <!-- xacro:us_sensor name="us_16" parent="base_link">
+    <origin xyz="0.230 0 0.300" rpy="0 3.14 3.14" />
+  </xacro:us_sensor-->
+      <!--Camera  -->
+<!-- <xacro:camera name="camera" parent="base_link">
+    <origin xyz="0 0 0.38" rpy="0 0 0" />
+  </xacro:camera>
+ -->
 </robot>

File: robot_model/mp_500/xacros/mp_500_body.xacro (robot description, xacro)
@@ -4,10 +4,10 @@
     <link name="${name}">
   <inertial>
-  <mass value="56.4" />
-  <origin xyz="0.000122063 0.106046383 0.229559509" rpy="0 0 0"/>
-  <inertia ixx="1934.300108107" ixy="-1.1189088783480243" ixz="-0.40794571883788144"
-           iyy="1331.584507173302" iyz="-53.61566974072236"
-           izz="2565.65991901786" />
-  </inertial>
+        <mass value="5" />
+        <origin xyz="0 0 0" rpy="0 0 0"/>
+        <inertia ixx="1.71402" ixy="0.0" ixz="0.0"
+                 iyy="0.8856" iyz="0.0"
+                 izz="2.5725" />
+</inertial>
   <visual name='body'>
   <origin xyz="0.0 0.0 0" rpy="0 0 1.570796" />
@@ -23,4 +23,13 @@
   </collision>
   </link>
+<gazebo reference="${name}_link">
+    <kp>1000.0</kp>
+    <kd>10.0</kd>
+    <mu1>200</mu1>
+    <mu2>100</mu2>
+    <fdir1>0.5 0 0</fdir1>
+    <maxVel>10.0</maxVel>
+    <minDepth>0.0005</minDepth>
+    </gazebo>
   </xacro:macro>
 </robot>

File: robot_model/mp_500/xacros/mp_500_caster_wheel.xacro (robot description, xacro)
@@ -4,15 +4,17 @@
    <joint name="${name}_joint" type="fixed">
     <insert_block name="origin" />
+        <axis xyz="0 -1 0" />
       <limit effort="1000.0" lower="-1e+16" upper="1e+16" velocity="3.5"/>
       <parent link="${parent}" />
       <child link="${name}_link" />
-      <joint_properties damping="1" friction="1" />
+      <joint_properties damping="1.0" friction="1.0" />
    </joint>
    <link name="${name}_link" type="wheel">
     <inertial>
-      <mass value="3.5" />
-      <origin xyz="0.000000010 -0.045437214 -0.073569633" rpy="0 0 0" />
-      <inertia ixx="13.177588678963057" ixy="-0.00000019386313414965295" ixz="-0.0000007636494859403484" iyy="8.48847991205267" iyz="-2.366298925984707" izz="7.157972023102095" />
-    </inertial>
+        <mass value="1.82362"/>
+        <inertia ixx="0.00499743171" ixy="0.00000004464" ixz="-0.00000002245"
+                 iyy="0.00499741733" iyz="0.00000000164"
+izz="0.00839239692"/>
+</inertial>
       <visual name='castor_wheel'>
     <origin xyz="0 0 0" rpy="0 0 0" />
@@ -28,4 +30,13 @@
     </collision>
 </link>
+<gazebo reference="${name}_link">
+      <kp>8000.0</kp>
+      <kd>1460.0</kd>
+      <mu1>0.5</mu1>
+      <mu2>0.2</mu2>
+      <fdir1>1 0 0</fdir1>
+      <maxVel>3.0</maxVel>
+      <minDepth>0.00</minDepth>
+</gazebo>
   </xacro:macro>
 </robot>

File: robot_model/mp_500/xacros/mp_500_gazebo.xacro (robot description, xacro)
@@ -1,16 +1,8 @@
 <?xml version="1.0"?>
 <robot name="mp_500" xmlns:xacro="http://www.ros.org/wiki/xacro">
-   <gazebo reference="base_link">
-    <gravity>true</gravity>
-    <self_collide>false</self_collide>
-  </gazebo>
-  <gazebo reference="castor_wheel_link">
-    <gravity>true</gravity>
-    <self_collide>false</self_collide>
-  </gazebo>
   <gazebo reference="lidar_1_link">
       <sensor type="ray" name="lidar_1_link">
           <pose>0 0 0 0 0 0</pose>
-          <visualize>true</visualize>
+          <visualize>false</visualize>
           <update_rate>40</update_rate>
           <ray>
@@ -39,17 +31,133 @@
           </ray>
           <plugin name="lidar_1_link" filename="libgazebo_ros_laser.so">
-            <topicName>sick/scan</topicName>
-            <frameName>laserscanner_1_link</frameName>
+            <topicName>lidar_1/scan_filtered</topicName>
+            <frameName>lidar_1_link</frameName>
           </plugin>
         </sensor>
   </gazebo>
+    <gazebo reference="imu_1_link">
+    <gravity>true</gravity>
+    <sensor name="imu_sensor" type="imu">
+      <always_on>true</always_on>
+      <update_rate>100</update_rate>
+      <visualize>true</visualize>
+      <topic>__default_topic__</topic>
+      <plugin filename="libgazebo_ros_imu_sensor.so" name="imu_plugin">
+        <topicName>imu</topicName>
+        <bodyName>imu_link</bodyName>
+        <updateRateHZ>10.0</updateRateHZ>
+        <gaussianNoise>0.0</gaussianNoise>
+        <xyzOffset>0 0 0</xyzOffset>
+        <rpyOffset>0 0 0</rpyOffset>
+        <frameName>imu_link</frameName>
+      </plugin>
+      <pose>0 0 0 0 0 0</pose>
+    </sensor>
+  </gazebo>
+  <gazebo reference="us_1_link">
+  <!-- Visuals / Collisions omitted for this example -->
+  <sensor type="ray" name="range">
+    <ray>
+         <scan>
+            <horizontal>
+               <samples>1</samples>
+               <resolution>1.0</resolution>
+               <min_angle>-0.01</min_angle>
+               <max_angle>0.01</max_angle>
+            </horizontal>
+            <vertical>
+               <samples>1</samples>
+               <resolution>1</resolution>
+               <min_angle>-0.01</min_angle>
+               <max_angle>0.01</max_angle>
+            </vertical>
+         </scan>
+         <range>
+            <min>0.01</min>
+            <max>3.75</max>
+            <resolution>0.02</resolution>
+         </range>
+      </ray>
+    <plugin name="libgazebo_ros_range" filename="libgazebo_ros_range.so">
+         <gaussianNoise>0.005</gaussianNoise>
+         <alwaysOn>true</alwaysOn>
+         <updateRate>50</updateRate>
+         <topicName>us_sensor</topicName>
+         <frameName>us_1_link</frameName>
+         <radiation>SONAR</radiation>
+         <fov>0.2967</fov>
+    </plugin>
+  </sensor>
+  </gazebo>
+    <!-- camera -->
+  <gazebo reference="camera_link">
+    <sensor type="camera" name="camera1">
+      <update_rate>30.0</update_rate>
+      <camera name="head">
+        <horizontal_fov>1.3962634</horizontal_fov>
+        <image>
+          <width>800</width>
+          <height>800</height>
+          <format>R8G8B8</format>
+        </image>
+        <clip>
+          <near>0.02</near>
+          <far>300</far>
+        </clip>
+        <noise>
+          <type>gaussian</type>
+          <!-- Noise is sampled independently per pixel on each frame.
+               That pixel's noise value is added to each of its color
+               channels, which at that point lie in the range [0,1]. -->
+          <mean>0.0</mean>
+          <stddev>0.007</stddev>
+        </noise>
+      </camera>
+      <plugin name="camera_controller" filename="libgazebo_ros_camera.so">
+        <alwaysOn>true</alwaysOn>
+        <updateRate>0.0</updateRate>
+        <cameraName>camera1</cameraName>
+        <imageTopicName>image_raw</imageTopicName>
+        <cameraInfoTopicName>camera_info</cameraInfoTopicName>
+        <frameName>camera_link</frameName>
+        <hackBaseline>0.07</hackBaseline>
+        <distortionK1>0.0</distortionK1>
+        <distortionK2>0.0</distortionK2>
+        <distortionK3>0.0</distortionK3>
+        <distortionT1>0.0</distortionT1>
+        <distortionT2>0.0</distortionT2>
+      </plugin>
+    </sensor>
+  </gazebo>
   <gazebo>
-    <plugin name="mp_500_controller" filename="libgazebo_ros_planar_move.so">
-      <commandTopic>cmd_vel</commandTopic>
-      <odometryTopic>odom</odometryTopic>
-      <odometryFrame>odom</odometryFrame>
-      <odometryRate>20.0</odometryRate>
-      <robotBaseFrame>base_link</robotBaseFrame>
+    <plugin name="diff_dirve_controller" filename="libgazebo_ros_diff_drive.so">
+        <alwaysOn>true</alwaysOn>
+        <updateRate>100</updateRate>
+        <legacyMode>false</legacyMode>
+        <torque>2.5</torque>
+        <leftJoint>wheel_left_joint</leftJoint>
+        <rightJoint>wheel_right_joint</rightJoint>
+        <wheelSeparation>0.592</wheelSeparation>
+        <wheelDiameter>0.260</wheelDiameter>
+        <commandTopic>cmd_vel</commandTopic>
+        <rosDebugLevel>na</rosDebugLevel>
+        <odometryTopic>odom</odometryTopic>
+        <odometryFrame>odom</odometryFrame>
+        <robotBaseFrame>base_link</robotBaseFrame>
+        <publishWheelTF>true</publishWheelTF>
+        <publishWheelJointState>true</publishWheelJointState>
+        <wheelAcceleration>0</wheelAcceleration>
+        <wheelTorque>200</wheelTorque>
+        <odometrySource>world</odometrySource>
+        <publishTf>1</publishTf>
+        <publishOdomTF>true</publishOdomTF>
     </plugin>
   </gazebo>
+<!-- <gazebo>
+  <plugin name="gazebo_ros_control" filename="libgazebo_ros_control.so">
+ <legacyModeNS> false </legacyModeNS>
+  <robotParam>/robot_description</robotParam>
+       <robotSimType>gazebo_ros_control/DefaultRobotHWSim</robotSimType>
+  </plugin>
+</gazebo> -->
 </robot>

Commit message: Robot models are updated and depreceated tags are removed

File: robot_model/mp_500/mp_500.urdf.xacro (robot description, xacro)
@@ -18,14 +18,17 @@
   <!-- <xacro:include filename="$(find neo_mp_500)/robot_model/mp_500/xacros/imu.xacro" />
   <xacro:include filename="$(find neo_mp_500)/robot_model/mp_500/xacros/ultrasonic.xacro" /> -->
-  <xacro:mp_500_base name="base_link">
+  <link name="base_link" />
+  <!-- Base link macro -->
+ <xacro:mp_500_base name="base_footprint" parent="base_link">
+    <origin xyz="0 0 0" rpy="0 0 0" />
   </xacro:mp_500_base>
   <!-- Wheel Macro -->
-  <xacro:caster_wheel name="caster_wheel" parent="base_link">
+  <xacro:caster_wheel name="caster_wheel" parent="base_footprint">
     <origin xyz="-0.43 0. 0.176" rpy="-1.570796 0 1.570796 " />
   </xacro:caster_wheel>
-  <xacro:fixed_wheel_right name="wheel_right" parent="base_link" number="1">
+  <xacro:fixed_wheel_right name="wheel_right" parent="base_footprint" number="1">
     <origin xyz="0. -0.25 0.13" rpy="0 0 -1.570796" />
   </xacro:fixed_wheel_right>
-  <xacro:fixed_wheel_left name="wheel_left" parent="base_link" number="2">
+  <xacro:fixed_wheel_left name="wheel_left" parent="base_footprint" number="2">
     <origin xyz="0. 0.25 0.13" rpy="0 0 -1.570796" />
   </xacro:fixed_wheel_left>

File: robot_model/mp_500/xacros/camera.xacro (robot description, xacro)
@@ -5,5 +5,5 @@
     <joint name="${name}_joint" type="fixed">
       <axis xyz="0 1 0" />
-      <insert_block name="origin" />
+      <xacro:insert_block name="origin" />
       <parent link="${parent}"/>
       <child link="${name}_link"/>

File: robot_model/mp_500/xacros/micro_scan.xacro (robot description, xacro)
@@ -4,5 +4,5 @@
     <joint name="${name}_joint" type="fixed">
       <axis xyz="0 1 0" />
-      <insert_block name="origin" />
+      <xacro:insert_block name="origin" />
       <parent link="${parent}"/>
       <child link="${name}_link"/>

File: robot_model/mp_500/xacros/mp_500_body.xacro (robot description, xacro)
@@ -1,6 +1,14 @@
 <?xml version="1.0"?>
 <robot xmlns:xacro="http://www.ros.org/wiki/xacro" name="mp_500">
-  <xacro:macro name="mp_500_base" params="name">
-    <link name="${name}">
+  <xacro:macro name="mp_500_base" params="name parent *origin">
+    <joint name="${name}_joint" type="fixed">
+      <xacro:insert_block name="origin" />
+      <axis xyz="0 0 -1" />
+      <!-- <limit effort="1000.0" lower="-1e+16" upper="1e+16" velocity="3.5"/> -->
+      <joint_properties damping="1" friction="1" />
+      <parent link="${parent}" />
+      <child link="${name}" />
+   </joint>
+  <link name="${name}">
   <inertial>
         <mass value="5" />
@@ -9,5 +17,5 @@
                  iyy="0.8856" iyz="0.0"
                  izz="2.5725" />
-</inertial>
+  </inertial>
   <visual name='body'>
   <origin xyz="0.0 0.0 0" rpy="0 0 1.570796" />

File: robot_model/mp_500/xacros/mp_500_caster_wheel.xacro (robot description, xacro)
@@ -3,5 +3,5 @@
   <xacro:macro name="caster_wheel" params="name parent *origin">
    <joint name="${name}_joint" type="fixed">
-    <insert_block name="origin" />
+    <xacro:insert_block name="origin" />
         <axis xyz="0 -1 0" />
       <limit effort="1000.0" lower="-1e+16" upper="1e+16" velocity="3.5"/>

File: robot_model/mp_500/xacros/mp_500_fixed_wheel.xacro (robot description, xacro)
@@ -3,5 +3,5 @@
   <xacro:macro name="fixed_wheel" params="name parent *origin">
    <joint name="${name}_joint" type="fixed">
-    <insert_block name="origin" />
+    <xacro:insert_block name="origin" />
     <axis xyz="0 1 0" />
     <joint_properties damping="1" friction="1" />

File: robot_model/mp_500/xacros/mp_500_fixed_wheel_left.xacro (robot description, xacro)
@@ -3,5 +3,5 @@
   <xacro:macro name="fixed_wheel_left" params="name parent number *origin">
     <joint name="${name}_joint" type="revolute">
-    <insert_block name="origin" />
+    <xacro:insert_block name="origin" />
     <limit effort="1000.0" lower="-1e+16" upper="1e+16" velocity="3.5"/>
     <axis xyz="-1 0 0" />

File: robot_model/mp_500/xacros/mp_500_fixed_wheel_right.xacro (robot description, xacro)
@@ -3,5 +3,5 @@
   <xacro:macro name="fixed_wheel_right" params="name parent number *origin">
     <joint name="${name}_joint" type="revolute">
-    <insert_block name="origin" />
+    <xacro:insert_block name="origin" />
     <limit effort="1000.0" lower="-1e+16" upper="1e+16" velocity="3.5"/>
     <axis xyz="-1 0 0" />

File: robot_model/mp_500/xacros/sick_S300.xacro (robot description, xacro)
@@ -4,5 +4,5 @@
     <joint name="${name}_joint" type="fixed">
       <axis xyz="0 1 0" />
-      <insert_block name="origin" />
+      <xacro:insert_block name="origin" />
       <parent link="${parent}"/>
       <child link="${name}_link"/>
